File: pcb/ai_ardushield_motor.brd (EAGLE design)
At the start: 68.6 x 53.3 mm, 41 parts, among them IC1 PCA9685, IC2 TB6612FNG, IC3 TB6612FNG, J1 1X02ST, J10 1X04, J12 1X02ST, J2 1X03, J3 1X03, J4 1X06, J5 1X08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

Commit message: Fixed a few minor warnings in the ERC.
Parts:
- JS1, JS2, JS3, JS4, JS5: value (none) -> 1X02-SJNO
Changed lines of the file:
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@@
 <setting verticaltext="up"/>
 </settings>
-<grid distance="5" unitdist="mil" unit="mil" style="lines" multiple="1" display="yes" altdistance="0.025" altunitdist="inch" altunit="inch"/>
+<grid distance="50" unitdist="mil" unit="mil" style="lines" multiple="1" display="yes" altdistance="0.025" altunitdist="inch" altunit="inch"/>
 <layers>
 <layer number="1" name="Top" color="4" fill="1" visible="yes" active="yes"/>
@@
 <attribute name="NAME" x="31.496" y="7.62" size="1.27" layer="25" font="vector" ratio="10" rot="R90"/>
 </element>
-<element name="JS1" library="Ai_Connectors" package="1X02-SJ-NO" value="" x="62.865" y="33.02" smashed="yes">
+<element name="JS1" library="Ai_Connectors" package="1X02-SJ-NO" value="1X02-SJNO" x="62.865" y="33.02" smashed="yes">
 <attribute name="NAME" x="61.595" y="32.385" size="1.27" layer="51"/>
 </element>
-<element name="JS2" library="Ai_Connectors" package="1X02-SJ-NO" value="" x="62.865" y="35.56" smashed="yes">
+<element name="JS2" library="Ai_Connectors" package="1X02-SJ-NO" value="1X02-SJNO" x="62.865" y="35.56" smashed="yes">
 <attribute name="NAME" x="61.595" y="34.925" size="1.27" layer="51"/>
 </element>
-<element name="JS3" library="Ai_Connectors" package="1X02-SJ-NO" value="" x="62.865" y="38.1" smashed="yes">
+<element name="JS3" library="Ai_Connectors" package="1X02-SJ-NO" value="1X02-SJNO" x="62.865" y="38.1" smashed="yes">
 <attribute name="NAME" x="61.595" y="37.465" size="1.27" layer="51"/>
 </element>
-<element name="JS4" library="Ai_Connectors" package="1X02-SJ-NO" value="" x="62.865" y="40.64" smashed="yes">
+<element name="JS4" library="Ai_Connectors" package="1X02-SJ-NO" value="1X02-SJNO" x="62.865" y="40.64" smashed="yes">
 <attribute name="NAME" x="61.595" y="40.005" size="1.27" layer="51"/>
 </element>
-<element name="JS5" library="Ai_Connectors" package="1X02-SJ-NO" value="" x="62.865" y="43.18" smashed="yes">
+<element name="JS5" library="Ai_Connectors" package="1X02-SJ-NO" value="1X02-SJNO" x="62.865" y="43.18" smashed="yes">
 <attribute name="NAME" x="61.595" y="42.545" size="1.27" layer="51"/>
 </element>

Commit message: changed the pcb dimension width.
Parts:
- U1: device Ai_Boards:UNOR3 -> Ai_Boards:UNOR3@1
Connections:
- removed net N$28: J7.4, U1.GND@3
- net GND: now also J7.4, U1.GND@3
Routing:
- net N$28: track 3.17 -> 0.00 mm
- net GND: track 145.7 -> 148.9 mm
Changed lines of the file:
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@@
 <grid distance="50" unitdist="mil" unit="mil" style="lines" multiple="1" display="yes" altdistance="0.025" altunitdist="inch" altunit="inch"/>
 <layers>
-<layer number="1" name="Top" color="4" fill="1" visible="yes" active="yes"/>
-<layer number="16" name="Bottom" color="1" fill="1" visible="yes" active="yes"/>
+<layer number="1" name="Top" color="4" fill="1" visible="no" active="yes"/>
+<layer number="16" name="Bottom" color="1" fill="1" visible="no" active="yes"/>
 <layer number="17" name="Pads" color="2" fill="1" visible="yes" active="yes"/>
 <layer number="18" name="Vias" color="2" fill="1" visible="yes" active="yes"/>
@@
 </autorouter>
 <elements>
-<element name="U1" library="Ai_Boards" package="UNOR3" value="ARDUINOUNOR3" x="0" y="0" smashed="yes"/>
+<element name="U1" library="Ai_Boards" package="UNOR3@1" value="ARDUINOUNOR3" x="0" y="0" smashed="yes"/>
 <element name="J4" library="Ai_Connectors" package="1X06" value="1X06" x="57.15" y="5.715" smashed="yes" rot="R180">
 <attribute name="NAME" x="64.135" y="3.175" size="1.27" layer="25" font="vector" ratio="10"/>
@@
 <wire x1="31.496" y1="10.922" x2="31.496" y2="16.002" width="0.254" layer="16"/>
 <wire x1="21.932" y1="16.256" x2="22.821" y2="17.145" width="0.254" layer="1"/>
+<contactref element="U1" pad="GND@3"/>
+<contactref element="J7" pad="4"/>
+<wire x1="26.67" y1="50.8" x2="26.67" y2="47.625" width="0.254" layer="16"/>
 </signal>
 <signal name="SCL">
@@
 <wire x1="24.13" y1="50.8" x2="24.13" y2="47.625" width="0.254" layer="16"/>
 </signal>
-<signal name="N$28">
-<contactref element="U1" pad="GND@3"/>
-<contactref element="J7" pad="4"/>
-<wire x1="26.67" y1="50.8" x2="26.67" y2="47.625" width="0.254" layer="16"/>
-</signal>
 <signal name="N$29">

Commit message: New version including detailed BOM
Parts:
- added J11, J13, J14, J15, J16, J17, J18, J19, J20, J21, J22: 1X06-PROTO, Ai_Connectors:1X06-NOFIRST
- added U$14: AI-LOGOL, Ai_Miscellany:AI-LOGO-L
- C1, C2, C3: device Ai_Passives:PANASONIC_C -> Ai_Passives:CAP-PANASONIC-C
- C4, C5, C6, C7, C8: device Ai_Passives:0603-CAP -> Ai_Passives:CAP-0603
- J10: value 1X04 -> 1X02ST; device Ai_Connectors:1X04 -> Ai_Connectors:1X02-ST
- J12: value 1X02ST -> 1X06-PROTO; device Ai_Connectors:1X02-ST -> Ai_Connectors:1X06-NOFIRST
- J2: value 1X03 -> 2X03; device Ai_Connectors:1X03 -> Ai_Connectors:2X03
- J3: value 1X03 -> 1X06; device Ai_Connectors:1X03 -> Ai_Connectors:1X06
- J4: value 1X06 -> 1X08; device Ai_Connectors:1X06 -> Ai_Connectors:1X08
- J6: value 1X08 -> 1X10; device Ai_Connectors:1X08 -> Ai_Connectors:1X10
- J7: value 1X10 -> 1X05ST; device Ai_Connectors:1X10 -> Ai_Connectors:1X05-ST
- J9: value 1X05ST -> 1X04; device Ai_Connectors:1X05-ST -> Ai_Connectors:1X04
- LED1: device Ai_LED:0603-LED -> Ai_LED:LED-0603
- R1: value 1k -> 1K; device Ai_Passives:0603-RES -> Ai_Passives:RES-0603
- R2, R3, R4, R5, R6, R7, R8: device Ai_Passives:0603-RES -> Ai_Passives:RES-0603
- SW1: value SW-SPST -> SW-SPSTSMD06X06; device Ai_Electromechanical:SPST-SMD -> Ai_Electromechanical:SPST-SMD06X06
- U1: device Ai_Boards:UNOR3@1 -> Ai_Boards:UNOR3
- moved J3 67.7 mm to (57.1, 5.71), turned to 180 degrees
- moved J8 61.0 mm to (3.81, 17.0), turned to 270 degrees
- moved J5 45.5 mm to (54.6, 47.6), turned to 0 degrees
- moved J7 44.0 mm to (64.8, 20.1), turned to 90 degrees
- moved J12 31.9 mm to (21.6, 35.1), turned to 90 degrees
- moved J10 28.1 mm to (16.8, 3.56), turned to 0 degrees
- moved J6 24.1 mm to (30.5, 47.6)
- moved J4 20.3 mm to (36.8, 5.71)
- moved J9 15.8 mm to (11.0, 31.1)
- moved C4 6.38 mm to (19.2, 11.4), turned to 180 degrees
- moved J2 1.27 mm to (6.86, 49.8)
- moved R1 0.56 mm to (19.2, 9.73)
- moved C3 0.46 mm to (23.7, 22.0)
- moved C5 0.26 mm to (27.2, 12.3)
Connections:
- net 3V3: now also J4.5; no longer J5.5
- net 5V: now also J2.3, J2.4, J4.4; no longer J2.2, J3.2, J5.4
- net GND: now also J10.2, J2.2, J4.2, J4.3, J6.4, J7.3; no longer J12.2, J3.1, J5.2, J5.3, J7.4, J9.3
- net N$1: now also J5.1; no longer J6.1
- net N$15: now also J4.7; no longer J5.7
- net N$16: now also J4.8; no longer J5.8
- net N$17: now also J5.3; no longer J6.3
- net N$18: now also J5.4; no longer J6.4
- net N$19: now also J5.5; no longer J6.5
- net N$2: now also J5.2; no longer J6.2
- net N$20: now also J5.6; no longer J6.6
- net N$21: now also J5.7; no longer J6.7
- net N$22: now also J5.8; no longer J6.8
- net N$23: now also J7.1; no longer J8.1
- net N$24: now also J7.2; no longer J8.2
- net N$27: now also J6.3; no longer J7.3
- net N$29: now also J6.5; no longer J7.5
- net N$30: now also J6.6; no longer J7.6
- net N$31: now also J6.7; no longer J7.7
- net N$32: now also J6.8; no longer J7.8
- net N$35: now also J7.4; no longer J8.4
- net N$36: now also J7.5; no longer J8.5
- net N$38: now also J8.1; no longer J9.1
- net N$39: now also J8.2; no longer J9.2
- net N$40: now also J8.4; no longer J9.4
- net N$41: now also J8.5; no longer J9.5
- net N$5: now also J3.3; no longer J4.3
- net N$6: now also J3.4; no longer J4.4
- net N$7: now also J3.5; no longer J4.5
- net N$8: now also J3.6; no longer J4.6
- net PWM0: now also J9.1; no longer J10.1
- net PWM1: now also J9.2; no longer J10.2
- net PWM14: now also J9.3; no longer J10.3
- net PWM15: now also J9.4; no longer J10.4
- net PWM16: now also J2.6, J6.10; no longer J3.3, J7.10
- net PWM17: now also J2.5, J6.9; no longer J2.3, J7.9
- net RESET: now also J4.6; no longer J5.6
- net SCL: now also J3.1, J6.1; no longer J4.1, J7.1
- net SDA: now also J3.2, J6.2; no longer J4.2, J7.2
- net VIN: now also J4.1; no longer J5.1
- net VMOTOR: now also J10.1; no longer J12.1
Routing:
- net GND: track 148.9 -> 79.6 mm, vias 11 -> 12
- net VCC: track 160.7 -> 169.7 mm
- net PWM14: track 31.7 -> 34.8 mm
- net RESET: track 63.4 -> 62.7 mm
- net N$4: track 5.98 -> 5.39 mm
- net VM: track 104.4 -> 104.0 mm, vias 3 -> 5

Commit message: Updated to use latest libraries.
Parts:
- removed SW1: SW-SPSTSMD06X06, Ai_Electromechanical:SPST-SMD06X06
- added S1: SW-SPSTSMD06X06, Ai_Electromechanical:SW-SPST-SMD06X06
Connections:
- net GND: now also S1.A@1, S1.A@2; no longer SW1.A@1, SW1.A@2
- net RESET: now also S1.B@1, S1.B@2; no longer SW1.B@1, SW1.B@2
Routing:
- net RESET: track 62.7 -> 65.8 mm
Changed lines of the file:
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@@
 <layer number="111" name="LPC17xx" color="7" fill="1" visible="yes" active="yes"/>
 <layer number="112" name="tSilk" color="7" fill="1" visible="yes" active="yes"/>
+<layer number="113" name="Route13" color="7" fill="1" visible="no" active="no"/>
 <layer number="116" name="Patch_BOT" color="9" fill="4" visible="no" active="yes"/>
+<layer number="117" name="mPads" color="7" fill="1" visible="no" active="no"/>
+<layer number="118" name="mVias" color="7" fill="1" visible="no" active="no"/>
+<layer number="119" name="mUnrouted" color="7" fill="1" visible="no" active="no"/>
+<layer number="120" name="mDimension" color="7" fill="1" visible="no" active="no"/>
 <layer number="121" name="_tsilk" color="7" fill="1" visible="no" active="yes"/>
 <layer number="122" name="_bsilk" color="7" fill="1" visible="no" active="yes"/>
@@
 <layer number="127" name="_tValues" color="7" fill="1" visible="yes" active="yes"/>
 <layer number="128" name="_bValues" color="7" fill="1" visible="yes" active="yes"/>
+<layer number="129" name="mtStop" color="7" fill="1" visible="no" active="no"/>
+<layer number="130" name="mbStop" color="7" fill="1" visible="no" active="no"/>
 <layer number="131" name="tAdjust" color="7" fill="1" visible="no" active="yes"/>
 <layer number="132" name="bAdjust" color="7" fill="1" visible="no" active="yes"/>
+<layer number="133" name="mtFinish" color="7" fill="1" visible="no" active="no"/>
+<layer number="134" name="mbFinish" color="7" fill="1" visible="no" active="no"/>
+<layer number="135" name="mtGlue" color="7" fill="1" visible="no" active="no"/>
+<layer number="136" name="mbGlue" color="7" fill="1" visible="no" active="no"/>
+<layer number="137" name="mtTest" color="7" fill="1" visible="no" active="no"/>
+<layer number="138" name="mbTest" color="7" fill="1" visible="no" active="no"/>
+<layer number="139" name="mtKeepout" color="7" fill="1" visible="no" active="no"/>
+<layer number="140" name="mbKeepout" color="7" fill="1" visible="no" active="no"/>
+<layer number="141" name="mtRestrict" color="7" fill="1" visible="no" active="no"/>
+<layer number="142" name="mbRestrict" color="7" fill="1" visible="no" active="no"/>
+<layer number="143" name="mvRestrict" color="7" fill="1" visible="no" active="no"/>
 <layer number="144" name="Drill_legend" color="7" fill="1" visible="no" active="yes"/>
+<layer number="145" name="mHoles" color="7" fill="1" visible="no" active="no"/>
+<layer number="146" name="mMilling" color="7" fill="1" visible="no" active="no"/>
+<layer number="147" name="mMeasures" color="7" fill="1" visible="no" active="no"/>
+<layer number="148" name="mDocument" color="7" fill="1" visible="no" active="no"/>
+<layer number="149" name="mReference" color="7" fill="1" visible="no" active="no"/>
 <layer number="150" name="Notes" color="7" fill="1" visible="no" active="yes"/>
 <layer number="151" name="HeatSink" color="7" fill="1" visible="no" active="yes"/>
@@
 <layer number="154" name="FabDoc2" color="2" fill="1" visible="no" active="no"/>
 <layer number="155" name="FabDoc3" color="7" fill="15" visible="no" active="no"/>
+<layer number="191" name="mNets" color="7" fill="1" visible="no" active="no"/>
+<layer number="192" name="mBusses" color="7" fill="1" visible="no" active="no"/>
+<layer number="193" name="mPins" color="7" fill="1" visible="no" active="no"/>
+<layer number="194" name="mSymbols" color="7" fill="1" visible="no" active="no"/>
+<layer number="195" name="mNames" color="7" fill="1" visible="no" active="no"/>
+<layer number="196" name="mValues" color="7" fill="1" visible="no" active="no"/>
 <layer number="199" name="Contour" color="7" fill="1" visible="no" active="yes"/>
 <layer number="200" name="200bmp" color="1" fill="10" visible="no" active="yes"/>
@@
 <attribute name="NAME" x="15.9258" y="39.3446" size="1.27" layer="25" ratio="15" rot="R180"/>
 </element>
-<element name="SW1" library="Ai_Electromechanical" package="SPST-SMD06X06" value="SW-SPSTSMD06X06" x="4.826" y="31.623" smashed="yes" rot="R270"/>
 <element name="Q1" library="Ai_DiscreteSemis" package="TO252" value="P-FET" x="7.112" y="4.064" smashed="yes" rot="R90">
 <attribute name="NAME" x="9.398" y="7.493" size="1.27" layer="25" ratio="15"/>
@@
 <element name="J21" library="Ai_Connectors" package="1X06-NOFIRST" value="1X06-PROTO" x="44.45" y="35.052" smashed="yes" rot="R90"/>
 <element name="J22" library="Ai_Connectors" package="1X06-NOFIRST" value="1X06-PROTO" x="46.99" y="35.052" smashed="yes" rot="R90"/>
+<element name="S1" library="Ai_Electromechanical" package="SW-SPST-SMD06X06" value="SW-SPSTSMD06X06" x="4.826" y="31.75" smashed="yes" rot="R90"/>
 </elements>
 <signals>
@@
 <contactref element="J1" pad="2"/>
 <contactref element="C1" pad="C"/>
-<contactref element="SW1" pad="A@1"/>
-<contactref element="SW1" pad="A@2"/>
 <contactref element="Q1" pad="G"/>
 <contactref element="J7" pad="3"/>
@@
 <via x="58.9026" y="30.5562" extent="1-16" drill="0.508"/>
 <via x="31.0896" y="11.0744" extent="1-16" drill="0.508"/>
+<contactref element="S1" pad="A@2"/>
+<contactref element="S1" pad="A@1"/>
 </signal>
 <signal name="SCL">
@@
 <contactref element="U1" pad="RESET"/>
 <contactref element="J4" pad="6"/>
-<contactref element="SW1" pad="B@1"/>
-<contactref element="SW1" pad="B@2"/>
 <wire x1="33.02" y1="2.54" x2="31.75" y2="1.27" width="0.4064" layer="16"/>
 <wire x1="31.75" y1="1.27" x2="9.398" y2="1.27" width="0.4064" layer="16"/>
@@
 <wire x1="8.636" y1="23.876" x2="7.112" y2="25.146" width="0.4064" layer="16"/>
 <via x="7.112" y="25.146" extent="1-16" drill="0.508"/>
-<wire x1="7.076" y1="35.598" x2="7.076" y2="27.648" width="0.4064" layer="1"/>
-<wire x1="7.112" y1="25.146" x2="7.112" y2="27.612" width="0.4064" layer="1"/>
-<wire x1="7.112" y1="27.612" x2="7.076" y2="27.648" width="0.4064" layer="1"/>
 <wire x1="33.02" y1="5.715" x2="33.02" y2="2.54" width="0.4064" layer="1"/>
+<contactref element="S1" pad="B@1"/>
+<contactref element="S1" pad="B@2"/>
+<wire x1="7.112" y1="25.146" x2="6.604" y2="25.146" width="0.4064" layer="1"/>
+<wire x1="6.604" y1="25.146" x2="4.064" y2="27.686" width="0.4064" layer="1"/>
+<wire x1="4.064" y1="27.686" x2="2.665" y2="27.686" width="0.4064" layer="1"/>
+<wire x1="2.665" y1="27.686" x2="2.576" y2="27.775" width="0.4064" layer="1"/>
+<wire x1="2.576" y1="35.725" x2="2.576" y2="27.775" width="0.4064" layer="1"/>
 </signal>
 <signal name="N$15">
