File: pcb/ai_ardushield_motor.sch (EAGLE design)
At the start: 53 parts, among them IC1 PCA9685, IC2 TB6612FNG, IC3 TB6612FNG, J1 1X02ST, J10 1X02ST, J11 1X06-PROTO, J12 1X06-PROTO, J13 1X06-PROTO, J14 1X06-PROTO, J15 1X06-PROTO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

Commit message: Updated to use latest libraries.
Parts:
- renumbered SW1 to S1
Connections:
- net GND: no longer S1.A@2
- net RESET: no longer S1.B@2
Changed lines of the file:
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@@
 <layer number="111" name="LPC17xx" color="7" fill="1" visible="yes" active="yes"/>
 <layer number="112" name="tSilk" color="7" fill="1" visible="yes" active="yes"/>
+<layer number="113" name="Route13" color="7" fill="1" visible="no" active="no"/>
 <layer number="116" name="Patch_BOT" color="9" fill="4" visible="no" active="yes"/>
+<layer number="117" name="mPads" color="7" fill="1" visible="no" active="no"/>
+<layer number="118" name="mVias" color="7" fill="1" visible="no" active="no"/>
+<layer number="119" name="mUnrouted" color="7" fill="1" visible="no" active="no"/>
+<layer number="120" name="mDimension" color="7" fill="1" visible="no" active="no"/>
 <layer number="121" name="_tsilk" color="7" fill="1" visible="no" active="yes"/>
 <layer number="122" name="_bsilk" color="7" fill="1" visible="no" active="yes"/>
@@
 <layer number="127" name="_tValues" color="7" fill="1" visible="yes" active="yes"/>
 <layer number="128" name="_bValues" color="7" fill="1" visible="yes" active="yes"/>
+<layer number="129" name="mtStop" color="7" fill="1" visible="no" active="no"/>
+<layer number="130" name="mbStop" color="7" fill="1" visible="no" active="no"/>
 <layer number="131" name="tAdjust" color="7" fill="1" visible="no" active="yes"/>
 <layer number="132" name="bAdjust" color="7" fill="1" visible="no" active="yes"/>
+<layer number="133" name="mtFinish" color="7" fill="1" visible="no" active="no"/>
+<layer number="134" name="mbFinish" color="7" fill="1" visible="no" active="no"/>
+<layer number="135" name="mtGlue" color="7" fill="1" visible="no" active="no"/>
+<layer number="136" name="mbGlue" color="7" fill="1" visible="no" active="no"/>
+<layer number="137" name="mtTest" color="7" fill="1" visible="no" active="no"/>
+<layer number="138" name="mbTest" color="7" fill="1" visible="no" active="no"/>
+<layer number="139" name="mtKeepout" color="7" fill="1" visible="no" active="no"/>
+<layer number="140" name="mbKeepout" color="7" fill="1" visible="no" active="no"/>
+<layer number="141" name="mtRestrict" color="7" fill="1" visible="no" active="no"/>
+<layer number="142" name="mbRestrict" color="7" fill="1" visible="no" active="no"/>
+<layer number="143" name="mvRestrict" color="7" fill="1" visible="no" active="no"/>
 <layer number="144" name="Drill_legend" color="7" fill="1" visible="no" active="yes"/>
+<layer number="145" name="mHoles" color="7" fill="1" visible="no" active="no"/>
+<layer number="146" name="mMilling" color="7" fill="1" visible="no" active="no"/>
+<layer number="147" name="mMeasures" color="7" fill="1" visible="no" active="no"/>
+<layer number="148" name="mDocument" color="7" fill="1" visible="no" active="no"/>
+<layer number="149" name="mReference" color="7" fill="1" visible="no" active="no"/>
 <layer number="150" name="Notes" color="7" fill="1" visible="no" active="yes"/>
 <layer number="151" name="HeatSink" color="7" fill="1" visible="no" active="yes"/>
@@
 <layer number="154" name="FabDoc2" color="2" fill="1" visible="no" active="no"/>
 <layer number="155" name="FabDoc3" color="7" fill="15" visible="no" active="no"/>
+<layer number="191" name="mNets" color="7" fill="1" visible="no" active="no"/>
+<layer number="192" name="mBusses" color="7" fill="1" visible="no" active="no"/>
+<layer number="193" name="mPins" color="7" fill="1" visible="no" active="no"/>
+<layer number="194" name="mSymbols" color="7" fill="1" visible="no" active="no"/>
+<layer number="195" name="mNames" color="7" fill="1" visible="no" active="no"/>
+<layer number="196" name="mValues" color="7" fill="1" visible="no" active="no"/>
 <layer number="199" name="Contour" color="7" fill="1" visible="no" active="yes"/>
 <layer number="200" name="200bmp" color="1" fill="10" visible="no" active="yes"/>
@@
 <part name="U$5" library="Ai_Power" deviceset="5V" device=""/>
 <part name="C1" library="Ai_Passives" deviceset="CAP-POL" device="PANASONIC-C" value="100uF"/>
-<part name="SW1" library="Ai_Electromechanical" deviceset="SW-SPST" device="SMD06X06"/>
 <part name="GND9" library="Ai_Power" deviceset="GND" device=""/>
 <part name="Q1" library="Ai_DiscreteSemis" deviceset="P-FET" device=""/>
@@
 <part name="J21" library="Ai_Connectors" deviceset="1X06-PROTO" device="" value="1X06-PROTO"/>
 <part name="J22" library="Ai_Connectors" deviceset="1X06-PROTO" device="" value="1X06-PROTO"/>
+<part name="S1" library="Ai_Electromechanical" deviceset="SW-SPST" device="SMD06X06"/>
 </parts>
 <sheets>
@@
 <instance part="U$5" gate="G$1" x="138.43" y="176.53"/>
 <instance part="C1" gate="G$1" x="13.97" y="35.56"/>
-<instance part="SW1" gate="G$1" x="17.78" y="13.97"/>
 <instance part="GND9" gate="GND" x="10.16" y="7.62"/>
 <instance part="Q1" gate="G$1" x="85.09" y="36.195"/>
@@
 <instance part="J21" gate="G$1" x="234.95" y="151.13" smashed="yes" rot="R270"/>
 <instance part="J22" gate="G$1" x="234.95" y="148.59" smashed="yes" rot="R270"/>
+<instance part="S1" gate="G$1" x="17.78" y="13.97"/>
 </instances>
 <busses>
@@
 </segment>
 <segment>
-<pinref part="SW1" gate="G$1" pin="B@1"/>
 <wire x1="22.86" y1="13.97" x2="25.4" y2="13.97" width="0.1524" layer="91"/>
-<pinref part="SW1" gate="G$1" pin="B@2"/>
-<wire x1="25.4" y1="13.97" x2="27.305" y2="13.97" width="0.1524" layer="91"/>
-<wire x1="22.86" y1="11.43" x2="25.4" y2="11.43" width="0.1524" layer="91"/>
-<wire x1="25.4" y1="11.43" x2="25.4" y2="13.97" width="0.1524" layer="91"/>
-<junction x="25.4" y="13.97"/>
-<label x="27.305" y="13.97" size="1.27" layer="95" ratio="15" xref="yes"/>
+<label x="25.4" y="13.97" size="1.27" layer="95" ratio="15" xref="yes"/>
+<pinref part="S1" gate="G$1" pin="B@1"/>
 </segment>
 </net>
@@
 </segment>
 <segment>
-<pinref part="SW1" gate="G$1" pin="A@1"/>
 <pinref part="GND9" gate="GND" pin="GND"/>
 <wire x1="12.7" y1="13.97" x2="10.16" y2="13.97" width="0.1524" layer="91"/>
-<wire x1="10.16" y1="13.97" x2="10.16" y2="11.43" width="0.1524" layer="91"/>
-<pinref part="SW1" gate="G$1" pin="A@2"/>
-<wire x1="10.16" y1="11.43" x2="10.16" y2="10.16" width="0.1524" layer="91"/>
-<wire x1="10.16" y1="11.43" x2="12.7" y2="11.43" width="0.1524" layer="91"/>
-<junction x="10.16" y="11.43"/>
-</segment>
-<segment>
+<wire x1="10.16" y1="13.97" x2="10.16" y2="10.16" width="0.1524" layer="91"/>
+<pinref part="S1" gate="G$1" pin="A@1"/>
+</segment>
+<segment>
